File: ergogen/output/pcbs/dyad-choc-v1.kicad_pcb (KiCad board)
At the start: 2 copper layers, 238.4 x 105.9 mm, 79 parts

Commit message: Iterating design
Parts:
- removed the ? at (327.3, 127.8)
- removed the ? at (108.7, 127.8)
- removed the ? at (321.7, 173.4)
- removed the ? at (114.3, 173.4)
- removed the REF** at (319.3, 193.3)
- added ?: , lib:niceview_headers, F.Cu at (326.7, 132.7)
- added ?: , lib:niceview_headers, F.Cu at (109.3, 132.7)
- added ?: , Button_Switch_SMD:SW_SPST_B3U-1000P, F.Cu at (321.5, 174.9)
- added ?: , Button_Switch_SMD:SW_SPST_B3U-1000P, F.Cu at (114.5, 174.9)
- added REF**: VIA-0.6mm, VIA-0.6mm, F.Cu at (331.7, 139.7)
- added REF**: VIA-0.6mm, VIA-0.6mm, F.Cu at (325.4, 142.9)
- added REF**: VIA-0.6mm, VIA-0.6mm, F.Cu at (330.7, 147.3)
- added REF**: VIA-0.6mm, VIA-0.6mm, F.Cu at (315.2, 174.2)
- added REF**: VIA-0.6mm, VIA-0.6mm, F.Cu at (311.9, 178.8)
- added REF**: VIA-0.6mm, VIA-0.6mm, F.Cu at (300.2, 153.6)
- added REF**: VIA-0.6mm, VIA-0.6mm, F.Cu at (282.7, 148.4)
- added REF**: VIA-0.6mm, VIA-0.6mm, F.Cu at (226.8, 151.8)
- added REF**: VIA-0.6mm, VIA-0.6mm, F.Cu at (247.8, 137.5)
- added REF**: VIA-0.6mm, VIA-0.6mm, F.Cu at (266.6, 131.7)
- added REF**: VIA-0.6mm, VIA-0.6mm, F.Cu at (313.5, 147.7)
- added REF**: VIA-0.6mm, VIA-0.6mm, F.Cu at (328.5, 139.3)
- added REF**: VIA-0.6mm, VIA-0.6mm, F.Cu at (314.1, 149.3)
- added REF**: VIA-0.6mm, VIA-0.6mm, F.Cu at (314.7, 150.9)
- added REF**: VIA-0.6mm, VIA-0.6mm, F.Cu at (115.8, 138.3)
- added REF**: VIA-0.6mm, VIA-0.6mm, F.Cu at (112.7, 138.7)
- added REF**: VIA-0.6mm, VIA-0.6mm, F.Cu at (114.1, 136.2)
- added REF**: VIA-0.6mm, VIA-0.6mm, F.Cu at (116.4, 154.9)
- added REF**: VIA-0.6mm, VIA-0.6mm, F.Cu at (114.6, 134.6)
- added REF**: VIA-0.6mm, VIA-0.6mm, F.Cu at (105.8, 146.0)
- added REF**: VIA-0.6mm, VIA-0.6mm, F.Cu at (108.6, 148.2)
- added REF**: VIA-0.6mm, VIA-0.6mm, F.Cu at (106.3, 135.6)
- added REF**: VIA-0.6mm, VIA-0.6mm, F.Cu at (330.5, 137.2)
- added REF**: VIA-0.6mm, VIA-0.6mm, F.Cu at (109.3, 135.3)
- added REF**: VIA-0.6mm, VIA-0.6mm, F.Cu at (110.6, 142.9)
- added REF**: VIA-0.6mm, VIA-0.6mm, F.Cu at (116.8, 145.8)
- added REF**: VIA-0.6mm, VIA-0.6mm, F.Cu at (108.1, 175.7)
- added REF**: VIA-0.6mm, VIA-0.6mm, F.Cu at (114.5, 185.3)
- added REF**: VIA-0.6mm, VIA-0.6mm, F.Cu at (129.3, 154.4)
- added REF**: VIA-0.6mm, VIA-0.6mm, F.Cu at (146.8, 149.2)
- added REF**: VIA-0.6mm, VIA-0.6mm, F.Cu at (202.8, 151.8)
- added REF**: VIA-0.6mm, VIA-0.6mm, F.Cu at (181.8, 138.3)
- added REF**: VIA-0.6mm, VIA-0.6mm, F.Cu at (162.9, 132.5)
- added REF**: VIA-0.6mm, VIA-0.6mm, F.Cu at (328.2, 155.9)
- added REF**: VIA-0.6mm, VIA-0.6mm, F.Cu at (140.8, 145.5)
- added REF**: VIA-0.6mm, VIA-0.6mm, F.Cu at (141.8, 146.9)
- added REF**: VIA-0.6mm, VIA-0.6mm, F.Cu at (142.8, 148.3)
- added REF**: VIA-0.6mm, VIA-0.6mm, F.Cu at (331.3, 135.8)
- added REF**: VIA-0.6mm, VIA-0.6mm, F.Cu at (320.1, 144.7)
- added REF**: VIA-0.6mm, VIA-0.6mm, F.Cu at (322.3, 147.5)
- added REF**: VIA-0.6mm, VIA-0.6mm, F.Cu at (323.1, 134.8)
- added REF**: VIA-0.6mm, VIA-0.6mm, F.Cu at (326.1, 135.2)
- moved D32 200.7 mm to (319.8, 192.2), turned to 56 degrees
- moved S32 195.1 mm to (313.5, 186.8), turned to -34 degrees
- moved D31 173.8 mm to (301.9, 180.2), turned to 68 degrees
- moved S31 167.5 mm to (294.7, 176.2), turned to -22 degrees
- moved D17 123.1 mm to (197.8, 144.0), turned to -90 degrees
- moved S17 116.8 mm to (206.0, 143.0), turned to 0 degrees
- moved D16 97.3 mm to (197.8, 161.0), turned to -90 degrees
- moved S16 90.3 mm to (206.0, 160.0), turned to 0 degrees
- moved D21 38.9 mm to (173.8, 114.3), turned to -83 degrees
- moved D24 38.9 mm to (154.9, 108.5), turned to -83 degrees
- moved D27 38.9 mm to (138.3, 120.6), turned to -83 degrees
- moved D30 38.9 mm to (120.8, 125.8), turned to -83 degrees
- moved D18 38.9 mm to (197.8, 127.0), turned to -90 degrees
- moved D25 34.9 mm to (142.4, 154.4), turned to -83 degrees
- moved D26 34.9 mm to (140.4, 137.5), turned to -83 degrees
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Connections:
- D1 pad 1: P8 -> ROW2
- D10 pad 1: P8 -> ROW2
- D11 pad 1: P7 -> ROW1
- D12 pad 1: P6 -> ROW0
- D13 pad 1: P8 -> ROW2
- D14 pad 1: P7 -> ROW1
- D15 pad 1: P6 -> ROW0
- D16 pad 1: P9 -> ROW2
- D16 pad 2: inner_sole -> mirror_pinky_bottom
- D17 pad 1: P9 -> ROW1
- D17 pad 2: outer_sole -> mirror_pinky_home
- D18 pad 1: P8 -> ROW0
- D18 pad 2: mirror_pinky_bottom -> mirror_pinky_top
- D19 pad 1: P7 -> ROW2
- D19 pad 2: mirror_pinky_home -> mirror_ring_bottom
- D2 pad 1: P7 -> ROW1
- D20 pad 1: P6 -> ROW1
- D20 pad 2: mirror_pinky_top -> mirror_ring_home
- D21 pad 1: P8 -> ROW0
- D21 pad 2: mirror_ring_bottom -> mirror_ring_top
- D22 pad 1: P7 -> ROW2
- D22 pad 2: mirror_ring_home -> mirror_middle_bottom
- D23 pad 1: P6 -> ROW1
- D23 pad 2: mirror_ring_top -> mirror_middle_home
- D24 pad 1: P8 -> ROW0
- D24 pad 2: mirror_middle_bottom -> mirror_middle_top
- D25 pad 1: P7 -> ROW2
- D25 pad 2: mirror_middle_home -> mirror_index_bottom
- D26 pad 1: P6 -> ROW1
- D26 pad 2: mirror_middle_top -> mirror_index_home
- D27 pad 1: P8 -> ROW0
- D27 pad 2: mirror_index_bottom -> mirror_index_top
- D28 pad 1: P7 -> ROW2
- D28 pad 2: mirror_index_home -> mirror_inner_bottom
- D29 pad 1: P6 -> ROW1
- D29 pad 2: mirror_index_top -> mirror_inner_home
- D3 pad 1: P6 -> ROW0
- D30 pad 1: P8 -> ROW0
- D30 pad 2: mirror_inner_bottom -> mirror_inner_top
- D31 pad 1: P7 -> ROW3
- D31 pad 2: mirror_inner_home -> inner_sole
- D32 pad 1: P6 -> ROW3
- D32 pad 2: mirror_inner_top -> outer_sole
- D33 pad 1: P9 -> ROW3
- D34 pad 1: P9 -> ROW3
- D4 pad 1: P8 -> ROW2
- D5 pad 1: P7 -> ROW1
- D6 pad 1: P6 -> ROW0
- D7 pad 1: P8 -> ROW2
- D8 pad 1: P7 -> ROW1
- D9 pad 1: P6 -> ROW0
- MCU1 pad 10: P14 -> COL2
- MCU1 pad 11: P16 -> COL3
- MCU1 pad 12: P10 -> COL4
- MCU1 pad 21: P6 -> ROW0
- MCU1 pad 22: P7 -> ROW1
- MCU1 pad 23: P8 -> ROW2
- MCU1 pad 24: P9 -> ROW3
- MCU1 pad 8: P18 -> COL0
- MCU1 pad 9: P15 -> COL1
- MCU2 pad 10: P14 -> COL2
- MCU2 pad 11: P16 -> COL3
- MCU2 pad 12: P10 -> COL4
- MCU2 pad 21: P6 -> ROW0
- MCU2 pad 22: P7 -> ROW1
- MCU2 pad 23: P8 -> ROW2
- MCU2 pad 24: P9 -> ROW3
- MCU2 pad 8: P18 -> COL0
- MCU2 pad 9: P15 -> COL1
- S1 pad 1: P18 -> COL0
- S10 pad 1: P16 -> COL3
- S11 pad 1: P16 -> COL3
- S12 pad 1: P16 -> COL3
- S13 pad 1: P10 -> COL4
- S14 pad 1: P10 -> COL4
- S15 pad 1: P10 -> COL4
- S16 pad 1: P16 -> COL0
- S16 pad 2: inner_sole -> mirror_pinky_bottom
- S17 pad 1: P10 -> COL0
- S17 pad 2: outer_sole -> mirror_pinky_home
- S18 pad 1: P18 -> COL0
- S18 pad 2: mirror_pinky_bottom -> mirror_pinky_top
- S19 pad 1: P18 -> COL1
- S19 pad 2: mirror_pinky_home -> mirror_ring_bottom
- S2 pad 1: P18 -> COL0
- S20 pad 1: P18 -> COL1
- S20 pad 2: mirror_pinky_top -> mirror_ring_home
- S21 pad 1: P15 -> COL1
- S21 pad 2: mirror_ring_bottom -> mirror_ring_top
- S22 pad 1: P15 -> COL2
- S22 pad 2: mirror_ring_home -> mirror_middle_bottom
- S23 pad 1: P15 -> COL2
- S23 pad 2: mirror_ring_top -> mirror_middle_home
- S24 pad 1: P14 -> COL2
- S24 pad 2: mirror_middle_bottom -> mirror_middle_top
- S25 pad 1: P14 -> COL3
- S25 pad 2: mirror_middle_home -> mirror_index_bottom
- S26 pad 1: P14 -> COL3
- S26 pad 2: mirror_middle_top -> mirror_index_home
- S27 pad 1: P16 -> COL3
- S27 pad 2: mirror_index_bottom -> mirror_index_top
- S28 pad 1: P16 -> COL4
- S28 pad 2: mirror_index_home -> mirror_inner_bottom
- S29 pad 1: P16 -> COL4
- S29 pad 2: mirror_index_top -> mirror_inner_home
- S3 pad 1: P18 -> COL0
- S30 pad 1: P10 -> COL4
- S30 pad 2: mirror_inner_bottom -> mirror_inner_top
- S31 pad 1: P10 -> COL3
- S31 pad 2: mirror_inner_home -> inner_sole
- S32 pad 1: P10 -> COL4
- S32 pad 2: mirror_inner_top -> outer_sole
- S33 pad 1: P16 -> COL3
- S34 pad 1: P10 -> COL4
- S4 pad 1: P15 -> COL1
- S5 pad 1: P15 -> COL1
- S6 pad 1: P15 -> COL1
- S7 pad 1: P14 -> COL2
- S8 pad 1: P14 -> COL2
- S9 pad 1: P14 -> COL2
- T2 pad 2: POSTIVE -> POSITIVE
Other:
- board size 238.4 x 105.9 mm -> 237.1 x 103.4 mm
