File: ergogen/output/pcbs/dyad-choc-v1-draft.kicad_pcb (KiCad board)
At the start: 2 copper layers, 117.6 x 96.6 mm, 84 parts

Commit message: reversable design
Parts:
- removed the REF** at (254.4, 129.5)
Routing:
- net COL2: track 128.0 -> 129.1 mm
- net COL1: track 141.4 -> 142.1 mm
